File: MCU logger.kicad_sch (KiCad schematic)
At the start: 25 parts, among them U1 24LC1025, U2 24LC1025, U3 DS1337S_, U4 ATMEGA328P-AU, Y1 16 MHz, Y2 32.768 KHz

Commit message: comments
Other:
- note added: "Connectors and mounting"
- note added: "EEPROM"
- note added: "MCU"
- note added: "Real time Clock"
Changed lines of the file:
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@@
 		(company "Rishikesh Sharma")
+	)
+	(rectangle
+		(start 38.1 37.465)
+		(end 137.795 81.915)
+		(stroke
+			(width 0)
+			(type default)
+		)
+		(fill
+			(type none)
+		)
+	)
+	(rectangle
+		(start 152.4 22.86)
+		(end 276.225 94.615)
+		(stroke
+			(width 0)
+			(type default)
+		)
+		(fill
+			(type none)
+		)
+	)
+	(rectangle
+		(start 131.445 96.52)
+		(end 220.98 142.875)
+		(stroke
+			(width 0)
+			(type default)
+		)
+		(fill
+			(type none)
+		)
+	)
+	(rectangle
+		(start 31.75 88.9)
+		(end 127 129.54)
+		(stroke
+			(width 0)
+			(type default)
+		)
+		(fill
+			(type none)
+		)
+	)
+	(text "MCU"
+		(exclude_from_sim no)
+		(at 156.21 20.32 0)
+		(effects
+			(font
+				(size 1.27 1.27)
+			)
+		)
+	)
+	(text "EEPROM"
+		(exclude_from_sim no)
+		(at 38.1 87.63 0)
+		(effects
+			(font
+				(size 1.27 1.27)
+			)
+		)
+	)
+	(text "Connectors and mounting"
+		(exclude_from_sim no)
+		(at 144.78 146.05 0)
+		(effects
+			(font
+				(size 1.27 1.27)
+			)
+		)
+	)
+	(text "Real time Clock"
+		(exclude_from_sim no)
+		(at 46.99 35.56 0)
+		(effects
+			(font
+				(size 1.27 1.27)
+			)
+		)
 	)
 	(junction
